File: cad/kicad/sensor_kit/cryoskills_sensor_kit.kicad_pcb (KiCad board)
At the start: 2 copper layers, 130 x 60 mm, 95 parts, among them J1 PWR_In, J10 QWIIC_I2C_2, J11 DS18B20, J12 SERIAL_BREAKOUT, J13 USB_B, J2 PWR_SENSE_Panel, J3 PWR_SENSE_Battery, J4 Adalogger_3V3, J5 Adalogger_VBUS, J6 Adalogger_RegulatorEN, J7 PT1000_RTD_WHEAT, J8 SPI_BREAKOUT, J9 QWIIC_I2C_1, SW1 SPDT Switch, SW2 SW_Push, U1 RFM96W, U2 INA3221, U3 TPS62932DRLR, U4 FT231XQ

Commit message: corrects MISO/MIMO silkscreen labels
Connections:
- J8 pad 3: /MOSI -> /MISO
- J8 pad 4: /MISO -> /MOSI
Routing:
- net /MOSI: track 44.2 -> 49.2 mm
- net /MISO: track 49.2 -> 44.2 mm
Changed lines of the file:
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@@
       (stroke (width 0.1) (type solid)) (layer "F.Fab"))
     (pad "1" thru_hole rect (at 0 0 90) (size 3 3) (drill 1.52) (layers "*.Cu" "*.Mask")
-      (net 3 "GND") (pinfunction "Pin_1") (pintype "passive"))
+      (net 3 "GND") (pinfunction "Pin_1") (pintype "passive") (zone_connect 1) (thermal_bridge_width 1) (thermal_gap 0.38))
     (pad "2" thru_hole circle (at 5.08 0 90) (size 3 3) (drill 1.52) (layers "*.Cu" "*.Mask")
       (net 12 "/V_BAT") (pinfunction "Pin_2") (pintype "passive"))
@@
       (net 76 "/ADC_RTDm") (pintype "passive"))
     (pad "2" thru_hole oval (at 5.08 0 180) (size 1.8 1.8) (drill 0.8) (layers "*.Cu" "*.Mask")
-      (net 3 "GND") (pintype "passive"))
+      (net 3 "GND") (pintype "passive") (zone_connect 1) (thermal_bridge_width 0.508) (thermal_gap 0.38))
     (model "${KICAD6_3DMODEL_DIR}/Resistor_THT.3dshapes/R_Axial_DIN0204_L3.6mm_D1.6mm_P5.08mm_Horizontal.wrl"
       (offset (xyz 0 0 0))
@@
       (net 4 "/SCK") (pinfunction "Pin_2") (pintype "passive"))
     (pad "3" thru_hole oval (at 0 5.08 270) (size 1.7 1.7) (drill 1) (layers "*.Cu" "*.Mask")
-      (net 5 "/MOSI") (pinfunction "Pin_3") (pintype "passive"))
+      (net 6 "/MISO") (pinfunction "Pin_3") (pintype "passive"))
     (pad "4" thru_hole oval (at 0 7.62 270) (size 1.7 1.7) (drill 1) (layers "*.Cu" "*.Mask")
-      (net 6 "/MISO") (pinfunction "Pin_4") (pintype "passive"))
+      (net 5 "/MOSI") (pinfunction "Pin_4") (pintype "passive"))
     (model "${KICAD6_3DMODEL_DIR}/Connector_PinHeader_2.54mm.3dshapes/PinHeader_1x04_P2.54mm_Vertical.wrl"
       (offset (xyz 0 0 0))
@@
       (net 13 "/VCC_3V3") (pinfunction "VIN") (pintype "power_in"))
     (pad "2" thru_hole circle (at -12.7 -7.62 90) (size 2 2) (drill 1) (layers "*.Cu" "*.Mask")
-      (net 3 "GND") (pinfunction "GND") (pintype "passive"))
+      (net 3 "GND") (pinfunction "GND") (pintype "passive") (zone_connect 1) (thermal_bridge_width 0.508) (thermal_gap 0.38))
     (pad "3" thru_hole circle (at -12.7 -5.08 90) (size 2 2) (drill 1) (layers "*.Cu" "*.Mask")
       (net 64 "/RADIO_EN") (pinfunction "EN") (pintype "input"))
@@
       (net 2 "/ADC_REF+") (pinfunction "AREF") (pintype "input"))
     (pad "4" thru_hole circle (at 0 7.62 180) (size 1.8 1.8) (drill 0.8) (layers "*.Cu" "*.Mask")
-      (net 3 "GND") (pinfunction "GND") (pintype "power_in"))
+      (net 3 "GND") (pinfunction "GND") (pintype "power_in") (zone_connect 1) (thermal_bridge_width 0.508) (thermal_gap 0.38))
     (pad "5" thru_hole circle (at 0 10.16 180) (size 1.8 1.8) (drill 0.8) (layers "*.Cu" "*.Mask")
       (net 57 "unconnected-(A1-DAC0{slash}A0-Pad5)") (pinfunction "DAC0/A0") (pintype "bidirectional+no_connect"))
@@
       (net 8 "/UART_TXuC") (pinfunction "TX/D1") (pintype "bidirectional"))
     (pad "16" thru_hole circle (at 0 38.1 180) (size 1.8 1.8) (drill 0.8) (layers "*.Cu" "*.Mask")
-      (net 3 "GND") (pinfunction "GND") (pintype "passive"))
+      (net 3 "GND") (pinfunction "GND") (pintype "passive") (zone_connect 1) (thermal_bridge_width 0.508) (thermal_gap 0.38))
     (pad "17" thru_hole circle (at 20.32 38.1 180) (size 1.8 1.8) (drill 0.8) (layers "*.Cu" "*.Mask")
       (net 9 "/SDA") (pinfunction "SDA/D20") (pintype "bidirectional"))
@@
     (pad "23" thru_hole circle (at 20.32 22.86 180) (size 1.8 1.8) (drill 0.8) (layers "*.Cu" "*.Mask")
       (net 2 "/ADC_REF+") (pinfunction "D11") (pintype "bidirectional"))
-    (pad "24" thru_hole circle (at 20.32 20.32 180) (size 1.8 1.8) (drill 0.8) (layers "*.Cu" "*.Mask")
+    (pad "24" thru_hole circle (at 20.32 20.32 180) (size 1.6 1.8) (drill 0.8) (layers "*.Cu" "*.Mask")
       (net 67 "unconnected-(A1-D12-Pad24)") (pinfunction "D12") (pintype "bidirectional+no_connect"))
-    (pad "25" thru_hole circle (at 20.32 17.78 180) (size 1.8 1.8) (drill 0.8) (layers "*.Cu" "*.Mask")
+    (pad "25" thru_hole circle (at 20.32 17.78 180) (size 1.6 1.8) (drill 0.8) (layers "*.Cu" "*.Mask")
       (net 68 "unconnected-(A1-D13-Pad25)") (pinfunction "D13") (pintype "bidirectional+no_connect"))
     (pad "26" thru_hole circle (at 20.32 15.24 180) (size 1.8 1.8) (drill 0.8) (layers "*.Cu" "*.Mask")
@@
       (net 77 "/ADC_RTDp") (pinfunction "Pin_1") (pintype "passive"))
     (pad "2" thru_hole circle (at 5.08 0 180) (size 3 3) (drill 1.52) (layers "*.Cu" "*.Mask")
-      (net 3 "GND") (pinfunction "Pin_2") (pintype "passive"))
+      (net 3 "GND") (pinfunction "Pin_2") (pintype "passive") (zone_connect 1) (thermal_bridge_width 1) (thermal_gap 0.38))
     (model "C:/data/components/3D/MP012059.stp"
       (offset (xyz -5.08 0 0))
@@
     )
     (stroke (width 0) (type solid)) (fill solid) (layer "F.SilkS"))
-  (gr_circle (center 160.3 107.8) (end 160.7 107.8)
+  (gr_circle (center 157.5 106.8) (end 157.591349 106.891349)
     (stroke (width 0.15) (type solid)) (fill solid) (layer "F.SilkS"))
   (gr_line (start 78.499999 81.999999) (end 78.5 85)
@@
     (effects (font (size 1 1) (thickness 0.2) bold) (justify left bottom))
   )
-  (gr_text "MOSI" (at 74 126.25 90) (layer "F.SilkS")
+  (gr_text "MISO" (at 74 126.25 90) (layer "F.SilkS")
     (effects (font (size 1 1) (thickness 0.2)) (justify right))
   )
@@
     (effects (font (size 1 1) (thickness 0.2) bold) (justify left))
   )
-  (gr_text "MISO\n" (at 71.5 126.25 90) (layer "F.SilkS")
+  (gr_text "MOSI" (at 71.5 126.25 90) (layer "F.SilkS")
     (effects (font (size 1 1) (thickness 0.2)) (justify right))
   )
@@
   (via (at 61 84.5) (size 1.6) (drill 0.8) (layers "F.Cu" "B.Cu") (free) (net 3))
   (via (at 111 127) (size 1.6) (drill 0.8) (layers "F.Cu" "B.Cu") (free) (net 3))
-  (via (at 102.5 124) (size 0.762) (drill 0.4064) (layers "F.Cu" "B.Cu") (free) (net 3))
+  (via (at 103.1 124.1) (size 0.762) (drill 0.4064) (layers "F.Cu" "B.Cu") (free) (net 3))
   (via (at 154.83 83) (size 1.6) (drill 0.8) (layers "F.Cu" "B.Cu") (free) (net 3))
   (via (at 163.5 88.5) (size 0.762) (drill 0.4064) (layers "F.Cu" "B.Cu") (free) (net 3))
@@
   (segment (start 79.66 107.84) (end 86.5 107.84) (width 0.508) (layer "F.Cu") (net 4))
   (segment (start 76.58 110.92) (end 79.66 107.84) (width 0.508) (layer "F.Cu") (net 4))
-  (segment (start 78.2 105.3) (end 86.5 105.3) (width 0.508) (layer "F.Cu") (net 5))
-  (segment (start 74.04 109.46) (end 78.2 105.3) (width 0.508) (layer "F.Cu") (net 5))
-  (segment (start 74.04 123) (end 74.04 109.46) (width 0.508) (layer "F.Cu") (net 5))
+  (segment (start 71.5 107) (end 71.5 123) (width 0.508) (layer "F.Cu") (net 5))
+  (segment (start 86.5 102.76) (end 75.74 102.76) (width 0.508) (layer "F.Cu") (net 5))
+  (segment (start 75.74 102.76) (end 71.5 107) (width 0.508) (layer "F.Cu") (net 5))
   (segment (start 95.5 110.95) (end 91.5 110.95) (width 0.508) (layer "F.Cu") (net 5))
   (via (at 91.5 110.95) (size 1.6) (drill 0.8) (layers "F.Cu" "B.Cu") (net 5))
@@
   (segment (start 91.5 104) (end 90.26 102.76) (width 0.508) (layer "B.Cu") (net 5))
   (segment (start 91.5 110.95) (end 91.5 104) (width 0.508) (layer "B.Cu") (net 5))
-  (segment (start 71.5 107) (end 71.5 123) (width 0.508) (layer "F.Cu") (net 6))
-  (segment (start 86.5 102.76) (end 75.74 102.76) (width 0.508) (layer "F.Cu") (net 6))
+  (segment (start 78.2 105.3) (end 86.5 105.3) (width 0.508) (layer "F.Cu") (net 6))
+  (segment (start 74.04 109.46) (end 78.2 105.3) (width 0.508) (layer "F.Cu") (net 6))
   (segment (start 90 113.43) (end 95.5 113.43) (width 0.508) (layer "F.Cu") (net 6))
-  (segment (start 75.74 102.76) (end 71.5 107) (width 0.508) (layer "F.Cu") (net 6))
+  (segment (start 74.04 123) (end 74.04 109.46) (width 0.508) (layer "F.Cu") (net 6))
   (via (at 90 113.43) (size 1.6) (drill 0.8) (layers "F.Cu" "B.Cu") (net 6))
   (segment (start 90 106.5) (end 88.8 105.3) (width 0.508) (layer "B.Cu") (net 6))
@@
   (segment (start 110.5 117) (end 110.5 111) (width 0.508) (layer "F.Cu") (net 66))
   (via (at 110.5 117) (size 1.6) (drill 0.8) (layers "F.Cu" "B.Cu") (net 66))
-  (segment (start 104.5 123) (end 98.5 123) (width 0.508) (layer "B.Cu") (net 66))
-  (segment (start 95.5 104) (end 91.72 100.22) (width 0.508) (layer "B.Cu") (net 66))
-  (segment (start 98.5 123) (end 95.5 120) (width 0.508) (layer "B.Cu") (net 66))
+  (segment (start 104.3 123.2) (end 98.7 123.2) (width 0.508) (layer "B.Cu") (net 66))
   (segment (start 91.72 100.22) (end 86.5 100.22) (width 0.508) (layer "B.Cu") (net 66))
   (segment (start 95.5 120) (end 95.5 104) (width 0.508) (layer "B.Cu") (net 66))
-  (segment (start 110.5 117) (end 104.5 123) (width 0.508) (layer "B.Cu") (net 66))
+  (segment (start 98.7 123.2) (end 95.5 120) (width 0.508) (layer "B.Cu") (net 66))
+  (segment (start 95.5 104) (end 91.72 100.22) (width 0.508) (layer "B.Cu") (net 66))
+  (segment (start 110.5 117) (end 104.3 123.2) (width 0.508) (layer "B.Cu") (net 66))
   (segment (start 125.9 94.25) (end 127.5 94.25) (width 0.508) (layer "F.Cu") (net 69))
   (segment (start 120.82 95.65) (end 124.5 95.65) (width 0.508) (layer "F.Cu") (net 69))
@@
         (xy 121.75 127.25)
         (xy 120.5 128.5)
-        (xy 105.2 128.5)
-        (xy 93.72 117.02)
+        (xy 104.8 128.5)
+        (xy 93.32 117.02)
         (xy 86.5 117.02)
         (xy 86.5 118.97)

Commit message: updates production files from sensor kit materials
Parts:
- moved C10 36.1 mm to (116.6, 75.1)
- moved C12 36.1 mm to (107.2, 58.0)
- moved C14 36.1 mm to (114.7, 54.9)
- moved C15 36.1 mm to (105.0, 62.0)
- moved C5 36.1 mm to (124.3, 67.2)
- moved C6 36.1 mm to (124.4, 65.2)
- moved D8 36.1 mm to (117.1, 67.4)
- moved FB1 36.1 mm to (114.7, 58.1)
- moved R20 36.1 mm to (113.8, 85.9)
- moved R36 36.1 mm to (110.0, 58.5)
- moved U4 36.1 mm to (109.7, 62.7)
- moved A1 36.1 mm to (70.5, 63.0)
- moved C1 36.1 mm to (126.7, 84.0)
- moved C11 36.1 mm to (111.7, 58.0)
- moved C13 36.1 mm to (111.3, 67.1)
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Other:
- board text added: "0"
- board text added: "0 mm"
- board text added: "0.01 mm"
- board text added: "0.02"
- board text added: "0.035 mm"
- board text added: "0.1524 mm / 0.1524 mm"
- board text added: "0.2540 mm"
- board text added: "1"
- board text added: "1.51 mm"
- board text added: "1.6000 mm"
- board text added: "130.0000 mm x 60.0000 mm"
- board text added: "2"
- board text added: "3.3"
- board text added: "4.5"
- board text added: "B.Cu"
- board text added: "B.Mask"
- board text added: "B.Paste"
- board text added: "B.Silkscreen"
- board text added: "BOARD CHARACTERISTICS"
- board text added: "Board Thickness:"
- board text added: "Board overall dimensions:"
- board text added: "Bottom Silk Screen"
- board text added: "Bottom Solder Mask"
- board text added: "Bottom Solder Paste"
- board text added: "Castellated pads:"
- board text added: "Color"
- board text added: "Copper Finish:"
- board text added: "Copper Layer Count:"
- board text added: "CryoSkills Sensor Kit"
- board text added: "Datalogger PCB"
- board text added: "Dielectric"
- board text added: "Edge card connectors:"
- board text added: "Epsilon R"
- board text added: "F.Cu"
- board text added: "F.Mask"
- board text added: "F.Paste"
- board text added: "F.Silkscreen"
- board text added: "FR4"
- board text added: "Impedance Control:"
- board text added: "Layer Name"
- board text added: "Loss Tangent"
- board text added: "Material"
- board text added: "Min hole diameter:"
- board text added: "Min track/spacing:"
- board text added: "No"
- board text added: "None"
- board text added: "Not specified"
- board text added: "Plated Board Edge:"
- board text added: "Thickness (mm)"
- board text added: "Top Silk Screen"
- board text added: "Top Solder Mask"
- board text added: "Top Solder Paste"
- board text added: "Type"
- board text added: "copper"
- board text added: "core"
