File: cad/kicad/sensor_kit/voltage_regulator.kicad_sch (KiCad schematic)
At the start: 11 parts, among them U1 TPS62932DRLR

Commit message: fixes MISO/MOSI on RFM96, swaps Dp/Dm on USB and makes pads for THT resistors bigger
Parts:
- added D8: NZH3V6B,115, Diode_SMD:D_SOD-123F, symbol Device:D_Zener
- C2: value 100nF -> 22uF; MftrPartNo GRM21BR61A226ME44L -> GRM21BR61A226ME51K; Placed (none) -> Yes; Supplier (none) -> Farnell; SupplierPartNo (none) -> 3581408
- C7: Manufacturer TDK -> Murata; MftrPartNo C2012X5R1V106K085AC -> GRM21BR6YA106KE43L; Placed (none) -> Yes; Supplier (none) -> Farnell; SupplierPartNo (none) -> 2611943
- C7: MftrPartNo CGA3E2X7R1H104K080AA -> CGA3E2X7R1H104K080AD; Placed (none) -> Yes; Supplier (none) -> Farnell; SupplierPartNo (none) -> 3416359
- C7: Manufacturer Murata -> Multicomp Pro; MftrPartNo GRM155R71A333KA01D -> MC0402B333K100CT; Placed (none) -> Yes; Supplier (none) -> Farnell; SupplierPartNo (none) -> 2627355
- C7: Manufacturer Murata -> Multicomp ro; MftrPartNo GRM155R71A104KA01D -> MC0402B104J100CT; Placed (none) -> Yes; Supplier (none) -> Farnell; SupplierPartNo (none) -> 2627341
- C8: MftrPartNo GRM1555C1E470JA01D -> C0402C470K5GACTU; Placed (none) -> Yes; Supplier (none) -> Farnell; SupplierPartNo (none) -> 2581031
- L1: MftrPartNo 1255AY-2R7N# -> 1255AY-2R7N=P3; Placed (none) -> Yes; Supplier (none) -> Farnell; SupplierPartNo (none) -> 2871550
- R21: footprint (none) -> Resistor_SMD:R_0402_1005Metric; Manufacturer (none) -> Multicomp Pro; MftrPartNo (none) -> MCWR04X1502FTL; Placed (none) -> Yes; Supplier (none) -> Farnell; SupplierPartNo (none) -> 2447112
- R22: footprint Capacitor_SMD:C_0603_1608Metric -> Resistor_SMD:R_0603_1608Metric; Manufacturer (none) -> Multicomp Pro; MftrPartNo (none) -> MCWR06X1002FTL; Placed (none) -> Yes; Supplier (none) -> Farnell; SupplierPartNo (none) -> 2447230
- R23: footprint Capacitor_SMD:C_0603_1608Metric -> Resistor_SMD:R_0603_1608Metric; Manufacturer (none) -> WALSIN; MftrPartNo (none) -> WR04X3092FTL; Placed (none) -> Yes; Supplier (none) -> Farnell; SupplierPartNo (none) -> 2670493
- U1: Arrow Part Number TPS62932DRLR -> (none); Arrow Price/Stock https://www.arrow.com/en/products/tps62932drlr/texas-instru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 -> (none); Manufacturer (none) -> Texas Instruments; Manufacturer_Name Texas Instruments -> (none); Manufacturer_Part_Number TPS62932DRLR -> (none); MftrPartNo (none) -> TPS62932DRLR; Mouser Part Number 595-TPS62932DRLR -> (none); Mouser Price/Stock https://www.mouser.co.uk/ProductDetail/Texas-Instruments/TP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 -> (none); Placed (none) -> Yes; Supplier (none) -> Digi-Key; SupplierPartNo (none) -> 296-TPS62932DRLRCT-ND
Connections:
- net GND: now also D8.2 (A)
- net Vout: now also D8.1 (K)
Other:
- note added: "3.6V zener clamp"

Commit message: updates production files from sensor kit materials
Other:
- company: (none) -> Cardiff University & CryoSkills Organising Committee
- title: (none) -> CryoSkills Sensor Kit
Changed lines of the file:
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@@
 (kicad_sch (version 20230121) (generator eeschema)
   (paper "A4")
+  (title_block
+    (title "CryoSkills Sensor Kit")
+    (company "Cardiff University & CryoSkills Organising Committee")
+    (comment 1 "Auth: J. D. Hawkins, L. Craw, M. Prior-Jones, E. Fisher")
+    (comment 2 "Contact: hawkinsj22@cardiff.ac.uk")
+  )
   (junction (at 199.39 99.06) (diameter 0) (color 0 0 0 0)
   )
